File: pcb/daughterboard.kicad_pcb (KiCad board)
At the start: 2 copper layers, 22 x 31.3 mm, 27 parts, among them J1 USB_C_Receptacle_USB2.0, J2 Conn_01x02_Female, J3 Conn_01x02_Female, J4 USB_C_Receptacle_USB2.0, J5 Conn_01x02_Female, J6 Conn_01x02_Female

Commit message: gnd routing
Routing:
- net GND: track 11.5 -> 40.8 mm
Changed lines of the file:
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@@
     (effects (font (size 0.8 0.8) (thickness 0.15)) (justify mirror))
   )
-  (gr_text "D-" (at 47.249823 101.250027 165) (layer "B.SilkS")
+  (gr_text "D-" (at 43.087792 103.500694 165) (layer "B.SilkS")
     (effects (font (size 0.8 0.8) (thickness 0.15)) (justify mirror))
   )
@@
     (effects (font (size 1.5 1.5) (thickness 0.2)) (justify mirror))
   )
-  (gr_text "D+" (at 45.787031 99.174333 165) (layer "B.SilkS")
+  (gr_text "D+" (at 41.625 101.425 165) (layer "B.SilkS")
     (effects (font (size 0.8 0.8) (thickness 0.15)) (justify mirror))
   )
@@
   (segment (start 28.728213 85.2) (end 27.262816 83.734603) (width 0.4) (layer "F.Cu") (net 1))
   (segment (start 38.012816 82.485) (end 38.035 82.485) (width 0.3) (layer "F.Cu") (net 1))
+  (segment (start 36.862659 98.558262) (end 37.658262 98.558262) (width 0.3) (layer "F.Cu") (net 1))
+  (segment (start 38.01 84.29) (end 38.925 83.375) (width 0.3) (layer "F.Cu") (net 1))
   (segment (start 31.622816 83.521891) (end 31.750425 83.6495) (width 0.3) (layer "F.Cu") (net 1))
   (segment (start 38.427007 101.242782) (end 38.427007 100.418914) (width 0.3) (layer "F.Cu") (net 1))
+  (segment (start 38.01 85.3) (end 38.01 84.29) (width 0.3) (layer "F.Cu") (net 1))
   (segment (start 30.4125 85.2) (end 28.728213 85.2) (width 0.4) (layer "F.Cu") (net 1))
   (segment (start 29.630639 98.752782) (end 28.712007 98.752782) (width 0.4) (layer "F.Cu") (net 1))
+  (segment (start 37.658262 98.558262) (end 38.768139 99.668139) (width 0.3) (layer "F.Cu") (net 1))
   (segment (start 31.737007 100.183914) (end 31.768139 100.152782) (width 0.3) (layer "F.Cu") (net 1))
   (segment (start 28.712007 98.752782) (end 27.387007 100.077782) (width 0.4) (layer "F.Cu") (net 1))
   (segment (start 31.622816 82.485) (end 31.622816 83.521891) (width 0.3) (layer "F.Cu") (net 1))
+  (segment (start 36.193139 99.227782) (end 36.862659 98.558262) (width 0.3) (layer "F.Cu") (net 1))
+  (segment (start 38.768139 99.668139) (end 38.768139 100.077782) (width 0.3) (layer "F.Cu") (net 1))
   (segment (start 38.427007 100.418914) (end 38.768139 100.077782) (width 0.3) (layer "F.Cu") (net 1))
   (via (at 31.750425 83.6495) (size 0.8) (drill 0.4) (layers "F.Cu" "B.Cu") (net 1))
@@
   (via (at 38.925 83.375) (size 0.8) (drill 0.4) (layers "F.Cu" "B.Cu") (net 1))
   (via (at 31.768139 100.152782) (size 0.8) (drill 0.4) (layers "F.Cu" "B.Cu") (net 1))
+  (segment (start 31.937353 83.462572) (end 31.750425 83.6495) (width 0.3) (layer "B.Cu") (net 1))
+  (segment (start 31.768139 100.152782) (end 31.850619 100.235262) (width 0.3) (layer "B.Cu") (net 1))
+  (segment (start 31.850619 100.235262) (end 38.610659 100.235262) (width 0.3) (layer "B.Cu") (net 1))
+  (segment (start 31.768139 100.152782) (end 31.693139 100.077782) (width 0.3) (layer "B.Cu") (net 1))
+  (segment (start 38.837428 83.462572) (end 31.937353 83.462572) (width 0.3) (layer "B.Cu") (net 1))
+  (segment (start 31.665322 83.734603) (end 27.262816 83.734603) (width 0.3) (layer "B.Cu") (net 1))
+  (segment (start 38.610659 100.235262) (end 38.768139 100.077782) (width 0.3) (layer "B.Cu") (net 1))
+  (segment (start 38.925 83.375) (end 38.837428 83.462572) (width 0.3) (layer "B.Cu") (net 1))
+  (segment (start 31.750425 83.6495) (end 31.665322 83.734603) (width 0.3) (layer "B.Cu") (net 1))
+  (segment (start 31.693139 100.077782) (end 27.387007 100.077782) (width 0.3) (layer "B.Cu") (net 1))
   (segment (start 30.642816 83.855316) (end 30.642816 81.76) (width 0.4) (layer "F.Cu") (net 2))
   (segment (start 31.9875 85.2) (end 30.642816 83.855316) (width 0.4) (layer "F.Cu") (net 2))

Commit message: silkscreen
Parts:
- added kibuzzard-6284F97C: G***, kibuzzard-6284F97C, F.Cu at (28.3, 90.8)
- added kibuzzard-6284F97C: G***, kibuzzard-6284F97C, F.Cu at (43.9, 101.2)
- added kibuzzard-6284F97C: G***, kibuzzard-6284F97C, F.Cu at (59.6, 101.2)
- added kibuzzard-6284F97C: G***, kibuzzard-6284F97C, F.Cu at (19.4, 88.2)
- added kibuzzard-6284F97C: G***, kibuzzard-6284F97C, F.Cu at (35.0, 98.6)
- added kibuzzard-6284F97C: G***, kibuzzard-6284F97C, F.Cu at (43.9, 106.5)
- added kibuzzard-6284F97C: G***, kibuzzard-6284F97C, F.Cu at (19.3, 103.9)
- added kibuzzard-6284F97C: G***, kibuzzard-6284F97C, F.Cu at (50.7, 98.6)
- added kibuzzard-6284F97C: G***, kibuzzard-6284F97C, F.Cu at (35.0, 103.9)
- added kibuzzard-6284F97C: G***, kibuzzard-6284F97C, F.Cu at (59.6, 106.5)
- added kibuzzard-6284F97C: G***, kibuzzard-6284F97C, F.Cu at (19.3, 98.6)
- added kibuzzard-6284F97C: G***, kibuzzard-6284F97C, F.Cu at (28.2, 106.5)
- added kibuzzard-6284F97C: G***, kibuzzard-6284F97C, F.Cu at (44.0, 96.1)
- added kibuzzard-6284F97C: G***, kibuzzard-6284F97C, F.Cu at (50.7, 103.9)
- added kibuzzard-6284F97C: G***, kibuzzard-6284F97C, F.Cu at (44.0, 90.8)
- added kibuzzard-6284F97C: G***, kibuzzard-6284F97C, F.Cu at (50.8, 93.5)
- added kibuzzard-6284F97C: G***, kibuzzard-6284F97C, F.Cu at (19.4, 93.5)
- added kibuzzard-6284F97C: G***, kibuzzard-6284F97C, F.Cu at (28.2, 101.2)
- added kibuzzard-6284F97C: G***, kibuzzard-6284F97C, F.Cu at (35.1, 93.5)
- added kibuzzard-6284F97C: G***, kibuzzard-6284F97C, F.Cu at (28.3, 96.1)
- added kibuzzard-6284F97C: G***, kibuzzard-6284F97C, F.Cu at (50.8, 88.2)
- added kibuzzard-6284F97C: G***, kibuzzard-6284F97C, F.Cu at (59.7, 96.1)
- added kibuzzard-6284F97C: G***, kibuzzard-6284F97C, F.Cu at (59.7, 90.8)
- added kibuzzard-6284F97C: G***, kibuzzard-6284F97C, F.Cu at (35.1, 88.2)
- moved kibuzzard-6284F97C 63.1 mm to (17.7, 83.1)
- moved kibuzzard-6284F97C 63.1 mm to (58.0, 80.4)
- moved kibuzzard-6284F97C 63.1 mm to (49.1, 77.8)
- moved kibuzzard-6284F97C 63.1 mm to (42.3, 80.4)
- moved kibuzzard-6284F97C 63.1 mm to (33.4, 83.1)
- moved kibuzzard-6284F97C 63.1 mm to (26.6, 80.4)
- moved kibuzzard-6284F97C 63.1 mm to (33.4, 77.8)
- moved kibuzzard-6284F97C 63.1 mm to (26.6, 85.7)
- moved kibuzzard-6284F97C 63.1 mm to (58.0, 85.7)
- moved kibuzzard-6284F97C 63.1 mm to (49.1, 83.1)
- moved kibuzzard-6284F97C 63.1 mm to (17.7, 77.8)
- moved kibuzzard-6284F97C 63.1 mm to (42.3, 85.7)
Routing:
- net GND: track 40.8 -> 58.4 mm
Other:
- board text added: "0.1a"
