File: pcb/0xB2.kicad_sch (KiCad schematic)
At the start: 54 parts, among them J1 USB_C_Receptacle_USB2.0, J10 RGB, J11 serial, J2 Conn_01x12, J3 Conn_01x05, J4 Conn_01x12, J5 Conn_01x02, J6 Ribbon, J7 Ribbon, J8 trackball, J9 Serial, SW1 SW_Push, SW2 SW_Push, SW3 SW_SPST, U1 RP2040, U2 GD25Q80CEIGR, U3 XC6210B332MR-G, Y1 Crystal_GND24

Commit message: remove small reset button
Parts:
- removed SW1: SW_Push, Button_Switch_SMD:SW_SPST_CK_KXT3, symbol Switch:SW_Push
Connections:
- net GND: now also SW3.1 (A); no longer SW3.2 (B)
- net ~{RESET}: now also SW3.2 (B); no longer SW3.1 (A)
Other:
- moved on the sheet: SW3
Changed lines of the file:
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@@
   (junction (at 53.34 36.83) (diameter 0) (color 0 0 0 0)
   )
+  (junction (at 40.005 172.72) (diameter 0) (color 0 0 0 0)
+  )
   (junction (at 46.99 127) (diameter 0) (color 0 0 0 0)
   )
@@
   (junction (at 160.02 38.1) (diameter 0) (color 0 0 0 0)
   )
-  (junction (at 40.005 172.72) (diameter 0) (color 0 0 0 0)
-  )
   (junction (at 33.02 113.03) (diameter 0) (color 0 0 0 0)
   )
@@
     (stroke (width 0) (type default) (color 0 0 0 0))
   )
-  (wire (pts (xy 40.005 184.15) (xy 40.005 186.69))
-    (stroke (width 0) (type default) (color 0 0 0 0))
-  )
   (wire (pts (xy 101.6 175.26) (xy 110.49 175.26))
     (stroke (width 0) (type default) (color 0 0 0 0))
@@
     (stroke (width 0) (type default) (color 0 0 0 0))
   )
-  (wire (pts (xy 40.005 172.72) (xy 40.005 173.99))
-    (stroke (width 0) (type default) (color 0 0 0 0))
-  )
   (wire (pts (xy 101.6 184.15) (xy 101.6 185.42))
     (stroke (width 0) (type default) (color 0 0 0 0))
@@
     (effects (font (size 1.27 1.27)) (justify right bottom))
   )
-  (label "~{RESET}" (at 410.21 30.48 180)
-    (effects (font (size 1.27 1.27)) (justify right bottom))
-  )
   (label "D9" (at 191.77 81.28 180)
     (effects (font (size 1.27 1.27)) (justify right bottom))
@@
     (pin "2")
   )
-  (symbol (lib_id "Switch:SW_SPST") (at 415.29 30.48 0) (unit 1)
+  (symbol (lib_id "Switch:SW_SPST") (at 40.005 177.8 90) (unit 1)
     (in_bom yes) (on_board yes)
-    (property "Reference" "SW3" (id 0) (at 415.29 24.13 0))
-    (property "Value" "SW_SPST" (id 1) (at 415.29 26.67 0))
-    (property "Footprint" "Library:PushSwitch" (id 2) (at 415.29 30.48 0)
+    (property "Reference" "SW3" (id 0) (at 33.655 177.8 0))
+    (property "Value" "SW_SPST" (id 1) (at 36.195 177.8 0))
+    (property "Footprint" "Library:PushSwitch" (id 2) (at 40.005 177.8 0)
       (effects (font (size 1.27 1.27)) hide)
     )
-    (property "Datasheet" "~" (id 3) (at 415.29 30.48 0)
+    (property "Datasheet" "~" (id 3) (at 40.005 177.8 0)
       (effects (font (size 1.27 1.27)) hide)
     )
@@
     (pin "2")
   )
-  (symbol (lib_id "power:GND") (at 40.005 186.69 0) (unit 1)
-    (in_bom yes) (on_board yes)
-    (property "Reference" "#PWR05" (id 0) (at 40.005 193.04 0)
-      (effects (font (size 1.27 1.27)) hide)
-    )
-    (property "Value" "GND" (id 1) (at 40.005 190.5 0))
-    (property "Footprint" "" (id 2) (at 40.005 186.69 0)
-      (effects (font (size 1.27 1.27)) hide)
-    )
-    (property "Datasheet" "" (id 3) (at 40.005 186.69 0)
-      (effects (font (size 1.27 1.27)) hide)
-    )
-    (pin "1")
-  )
   (symbol (lib_id "Device:R") (at 198.12 126.365 180) (unit 1)
     (in_bom yes) (on_board yes)
@@
   (symbol (lib_id "power:+3.3V") (at 483.235 54.61 90) (unit 1)
     (in_bom yes) (on_board yes)
-    (property "Reference" "#PWR?" (id 0) (at 487.045 54.61 0)
+    (property "Reference" "#PWR0104" (id 0) (at 487.045 54.61 0)
       (effects (font (size 1.27 1.27)) hide)
     )
@@
     (pin "1")
   )
-  (symbol (lib_id "power:GND") (at 420.37 30.48 90) (unit 1)
+  (symbol (lib_id "power:GND") (at 40.005 182.88 0) (unit 1)
     (in_bom yes) (on_board yes)
-    (property "Reference" "#PWR043" (id 0) (at 426.72 30.48 0)
+    (property "Reference" "#PWR043" (id 0) (at 40.005 189.23 0)
       (effects (font (size 1.27 1.27)) hide)
     )
-    (property "Value" "GND" (id 1) (at 427.3549 30.636 90)
+    (property "Value" "GND" (id 1) (at 39.849 189.8649 90)
       (effects (font (size 1.27 1.27)) (justify left))
     )
-    (property "Footprint" "" (id 2) (at 420.37 30.48 0)
+    (property "Footprint" "" (id 2) (at 40.005 182.88 0)
       (effects (font (size 1.27 1.27)) hide)
     )
-    (property "Datasheet" "" (id 3) (at 420.37 30.48 0)
+    (property "Datasheet" "" (id 3) (at 40.005 182.88 0)
       (effects (font (size 1.27 1.27)) hide)
     )
@@
     (pin "2")
   )
-  (symbol (lib_id "Switch:SW_Push") (at 40.005 179.07 90) (unit 1)
-    (in_bom yes) (on_board yes) (fields_autoplaced)
-    (property "Reference" "SW1" (id 0) (at 41.275 177.7999 90)
-      (effects (font (size 1.27 1.27)) (justify right))
-    )
-    (property "Value" "SW_Push" (id 1) (at 41.275 180.3399 90)
-      (effects (font (size 1.27 1.27)) (justify right))
-    )
-    (property "Footprint" "Button_Switch_SMD:SW_SPST_CK_KXT3" (id 2) (at 34.925 179.07 0)
-      (effects (font (size 1.27 1.27)) hide)
-    )
-    (property "Datasheet" "~" (id 3) (at 34.925 179.07 0)
-      (effects (font (size 1.27 1.27)) hide)
-    )
-    (property "LCSC" "C319433" (id 4) (at 40.005 179.07 0)
-      (effects (font (size 1.27 1.27)) hide)
-    )
-    (pin "1")
-    (pin "2")
-  )
   (symbol (lib_id "Connector_Generic:Conn_01x12") (at 269.24 54.61 0) (mirror x) (unit 1)
     (in_bom no) (on_board yes)
@@
       (reference "#PWR04") (unit 1) (value "+3.3V") (footprint "")
     )
-    (path "/4f8a166b-9702-4d80-b4fa-22089550ab5e"
-      (reference "#PWR05") (unit 1) (value "GND") (footprint "")
-    )
     (path "/d17eab26-feb4-4974-b911-181dda768f7a"
       (reference "#PWR06") (unit 1) (value "GND") (footprint "")
@@
       (reference "#PWR0103") (unit 1) (value "+5V") (footprint "")
     )
+    (path "/660cfbd8-c920-41f3-b80c-7bd72ed4ad19"
+      (reference "#PWR0104") (unit 1) (value "+3.3V") (footprint "")
+    )
     (path "/e8bfe983-bddc-4d18-b952-2e1ab119dff0"
       (reference "#PWR0105") (unit 1) (value "+3.3V") (footprint "")
@@
       (reference "#PWR0106") (unit 1) (value "+3.3V") (footprint "")
     )
-    (path "/660cfbd8-c920-41f3-b80c-7bd72ed4ad19"
-      (reference "#PWR?") (unit 1) (value "+3.3V") (footprint "")
-    )
     (path "/4a21e78b-0ab0-4b88-8132-9b174e045719"
       (reference "C1") (unit 1) (value "1µ") (footprint "Capacitor_SMD:C_0603_1608Metric")
@@
       (reference "R14") (unit 1) (value "5.1k") (footprint "Resistor_SMD:R_0402_1005Metric")
     )
-    (path "/c30a3276-ac5c-4a68-880e-26478e1b53e4"
-      (reference "SW1") (unit 1) (value "SW_Push") (footprint "Button_Switch_SMD:SW_SPST_CK_KXT3")
-    )
     (path "/4ea9bd29-a5a9-4d62-b350-c59ad41d14d5"

Commit message: daughterboard work
Parts:
- added J12, J13, J14, J15: Conn_01x02_Female, Library:PinHeader_1x02_P2.54mm_Vertical, symbol Connector:Conn_01x02_Female
Connections:
- net D+: now also J15.2 (Pin_2); no longer J1.A6 (D+), J1.B6 (D+)
- net D-: now also J15.1 (Pin_1); no longer J1.A7 (D-), J1.B7 (D-)
- net GND: now also J12.2 (Pin_2), J14.1 (Pin_1)
- net VBUS: now also J14.2 (Pin_2); no longer J1.A4 (VBUS), J1.A9 (VBUS), J1.B4 (VBUS), J1.B9 (VBUS)
- new net: J1.A4 (VBUS), J1.A9 (VBUS), J1.B4 (VBUS), J1.B9 (VBUS), J12.1 (Pin_1)
- new net: J1.A6 (D+), J1.B6 (D+), J13.2 (Pin_2)
- new net: J1.A7 (D-), J1.B7 (D-), J13.1 (Pin_1)
Other:
- note added: "USB-C daughterboard"
- note removed: "USB-C connector"
- moved on the sheet: D2, F1, J9

Commit message: cleanup
Parts:
- removed FB1: FerriteBead_Small, Inductor_SMD:L_0603_1608Metric, symbol Device:FerriteBead_Small
- removed J1: USB_C_Receptacle_USB2.0, 0xLib_USB_Type-C:USB_C_Receptacle_HRO_TYPE-C-31-M-14, symbol Connector:USB_C_Receptacle_USB2.0
- removed J12, J13: Conn_01x02_Female, Library:PinHeader_1x02_P2.54mm_Vertical, symbol Connector:Conn_01x02_Female
- removed R4, R5: 5.1k, Resistor_SMD:R_0402_1005Metric, symbol Device:R
Connections:
- no-connect marks 10 -> 8
Other:
- note removed: "USB-C daughterboard"

Commit message: move daughterboard to its own repo
Parts:
- JP1, JP2: footprint (none) -> Library:SolderJumper-2_P1.3mm_Open_RoundedPad1.0x1.5mm
Changed lines of the file:
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@@
     (property "Reference" "JP1" (id 0) (at 453.39 43.18 0))
     (property "Value" "Jumper_2_Open" (id 1) (at 453.39 45.72 0))
-    (property "Footprint" "" (id 2) (at 453.39 49.53 0)
+    (property "Footprint" "Library:SolderJumper-2_P1.3mm_Open_RoundedPad1.0x1.5mm" (id 2) (at 453.39 49.53 0)
       (effects (font (size 1.27 1.27)) hide)
     )
@@
     (property "Reference" "JP2" (id 0) (at 453.39 52.705 0))
     (property "Value" "Jumper_2_Open" (id 1) (at 453.39 55.245 0))
-    (property "Footprint" "" (id 2) (at 453.39 59.055 0)
+    (property "Footprint" "Library:SolderJumper-2_P1.3mm_Open_RoundedPad1.0x1.5mm" (id 2) (at 453.39 59.055 0)
       (effects (font (size 1.27 1.27)) hide)
     )
@@
     )
     (path "/6cbb1601-aee9-4b85-b6c4-65af6cce90fe"
-      (reference "JP1") (unit 1) (value "Jumper_2_Open") (footprint "")
+      (reference "JP1") (unit 1) (value "Jumper_2_Open") (footprint "Library:SolderJumper-2_P1.3mm_Open_RoundedPad1.0x1.5mm")
     )
     (path "/e6e604e3-e924-4286-a2fc-11cd9fe47f3f"
-      (reference "JP2") (unit 1) (value "Jumper_2_Open") (footprint "")
+      (reference "JP2") (unit 1) (value "Jumper_2_Open") (footprint "Library:SolderJumper-2_P1.3mm_Open_RoundedPad1.0x1.5mm")
     )
     (path "/81213cff-519c-4fcf-ae25-6fad0fc859bb"
